Commit message: Added a new URDF with 0.5m long connections and a 500g foot piece

File: urdf/TorquePoleLong/urdf/TorquePoleLong.urdf (robot description, URDF)
Before this commit: robot TorquePole, 2 links, 1 joints
Links:
- link base_link: mass 0.36224 -> 0.36931; geometry collision mesh filename=package://TorquePoleLong/meshes/base_link.STL; visual mesh filename=package://TorquePoleLong/meshes/base_link.STL
- link pendulum: mass 0.066367 -> 0.073435; geometry collision mesh filename=package://TorquePoleLong/meshes/pendulum.STL; visual mesh filename=package://TorquePoleLong/meshes/pendulum.STL
Joints:
- joint PullyJoint: limit lower=6.28 upper=-1.57 effort=3 velocity=300 -> lower=-1.35 upper=4.5 effort=3 velocity=60
