Commit message: Second attempt...

File: urdf/TorquePole2/urdf/TorquePole2.urdf (robot description, URDF)
Before this commit: robot TorquePole2, 2 links, 1 joints
Links:
- link base_link: mass 0.13052 -> 0.130519789197275
- link pendulum_link: mass 0.027671 -> 0.091873

Commit message: Flipped the pole orientation to upward

File: urdf/TorquePole2/urdf/TorquePole2.urdf (robot description, URDF)
Before this commit: robot TorquePole2, 2 links, 1 joints
Links:
- link pendulum_link: mass 0.091873 -> 0.0918727464707182
