Commit message: The NN + Motor driver worked beautifully. Ready for the writeup. Updated URDF again, was thinking of trying some parameter randomization for a more robust policy.

File: urdf/TorquePole/urdf/TorquePole.urdf (robot description, URDF)
Before this commit: robot TorquePole, 2 links, 1 joints
Links:
- removed link pendulum
- added link pendulum_link, mass 0.098923; collision mesh filename=package://TorquePole/meshes/pendulum_link.STL; visual mesh filename=package://TorquePole/meshes/pendulum_link.STL
- link base_link: mass 0.36224 -> 0.18536
Joints:
- removed joint PullyJoint
- added joint pendulum: type continuous, parent base_link, child pendulum_link, origin xyz=0 0 0 rpy=0 0 0, axis 0 0 -1, limit effort=0.5 velocity=3000
