Commit message: Learned a new policy with the current hardware setup, time to test on HW

File: isaac/IsaacGymEnvs/assets/urdf/TorquePole/urdf/TorquePole.urdf (robot description, URDF)
Before this commit: robot TorquePole, 2 links, 1 joints
Links:
- link base_link: mass 0.130519789197275 -> 0.18536
- link pendulum_link: mass 0.091873 -> 0.098923
