Commit message: Reward function improved. Reward is now set to zero when touching the ground. Reward per time step when off the ground is the max achieved height since the foot left the ground. This promote high jumping and long air time behavior

File: isaac/IsaacGymEnvs/assets/urdf/Jumpy/urdf/Jumpy.urdf (robot description, URDF)
Before this commit: robot Jumpy, 4 links, 3 joints
Joints:
- joint Prismatic1: limit lower=-0.5 upper=0.5 effort=0 velocity=0 -> lower=-0.5 upper=1.5 effort=0 velocity=0
