Commit message: Updated Quad urdf

File: urdf/Quad/urdf/Quad.urdf (robot description, URDF)
Before this commit: robot Quad, 13 links, 12 joints
Links:
- link BL_Hip: mass 0 -> 0.244991783639187
- link Body: mass 7.9384 -> 7.93838617368297
- link FR_Hip: mass 0.24499 -> 0.244991783639187
Joints:
- joint BL_J1: axis 0 0 1 -> 0 0 -1; origin xyz=0 0 0 rpy=0 0 0 -> xyz=0.1 0.05 -0.205567 rpy=3.14159265358979 0 1.5707963267949
- joint BL_J2: axis -1 0 0 -> 0 0 -1; origin xyz=0 0 0 rpy=0 0 0 -> xyz=0 0.0700000000000002 0.045979703345944 rpy=1.5707963267949 -1.5707963267949 0
- joint BL_J3: axis 1 0 0 -> 0 0 1; origin xyz=0 0 0 rpy=0 0 0 -> xyz=0.318 0 0 rpy=0 0 0
- joint BR_J1: axis 0 0 1 -> 0 0 -1; origin xyz=0 0 0 rpy=0 0 0 -> xyz=-0.1 0.05 -0.20557 rpy=3.1416 0 -1.5708
- joint BR_J2: axis 1 0 0 -> 0 0 -1; origin xyz=0 0 0 rpy=0 0 0 -> xyz=0 0.0700000000000001 0.045979703345944 rpy=1.5707963267949 -1.5707963267949 0
- joint BR_J3: axis -1 0 0 -> 0 0 1; origin xyz=0 0 0 rpy=0 0 0 -> xyz=0.318 0 0 rpy=0 0 0
- joint FL_J1: origin xyz=0 0 0 rpy=0 0 0 -> xyz=0.1 0.05 0.20557 rpy=0 0 -1.5708
- joint FL_J2: axis -1 0 0 -> 0 0 -1; origin xyz=0 0 0 rpy=0 0 0 -> xyz=0 0.0700000000000001 0.045979703345944 rpy=1.5707963267949 -1.5707963267949 0
- joint FL_J3: axis 1 0 0 -> 0 0 1; origin xyz=0 0 0 rpy=0 0 0 -> xyz=0.318 0 0 rpy=0 0 0
- joint FR_J1: axis 0 0 1 -> 0 0 -1; origin xyz=0 0 0 rpy=0 0 0 -> xyz=-0.1 0.05 0.20557 rpy=0 0 1.5708
- joint FR_J2: axis 1 0 0 -> 0 0 -1; origin xyz=0 0 0 rpy=0 0 0 -> xyz=0 0.07 0.04598 rpy=1.5708 -1.5708 0
- joint FR_J3: axis -1 0 0 -> 0 0 1; origin xyz=0 0 0 rpy=0 0 0 -> xyz=0.318 0 0 rpy=0 0 0

Commit message: Did redoing all the reference axis and coords help?

File: urdf/Quad/urdf/Quad.urdf (robot description, URDF)
Before this commit: robot Quad, 13 links, 12 joints
Joints:
- joint BL_J1: axis 0 0 -1 -> 0 0 1; origin xyz=0.1 0.05 -0.205567 rpy=3.14159265358979 0 1.5707963267949 -> xyz=0.1 0.05 -0.205567 rpy=0 0 0
- joint BL_J2: axis 0 0 -1 -> -1 0 0; origin xyz=0 0.0700000000000002 0.045979703345944 rpy=1.5707963267949 -1.5707963267949 0 -> xyz=0.0700000000000002 0 -0.045979703345944 rpy=0 0 0
- joint BL_J3: axis 0 0 1 -> 1 0 0; origin xyz=0.318 0 0 rpy=0 0 0 -> xyz=0 0 -0.318 rpy=0 0 0
- joint BR_J1: axis 0 0 -1 -> 0 0 1; origin xyz=-0.1 0.05 -0.20557 rpy=3.1416 0 -1.5708 -> xyz=-0.1 0.0500000000000001 -0.205567 rpy=0 0 0
- joint BR_J2: axis 0 0 -1 -> 1 0 0; origin xyz=0 0.0700000000000001 0.045979703345944 rpy=1.5707963267949 -1.5707963267949 0 -> xyz=-0.0700000000000003 0 -0.045979703345944 rpy=0 0 0
- joint BR_J3: axis 0 0 1 -> -1 0 0; origin xyz=0.318 0 0 rpy=0 0 0 -> xyz=0 0 -0.318 rpy=0 0 0
- joint FL_J1: origin xyz=0.1 0.05 0.20557 rpy=0 0 -1.5708 -> xyz=0.1 0.05 0.205567 rpy=0 0 0
- joint FL_J2: axis 0 0 -1 -> -1 0 0; origin xyz=0 0.0700000000000001 0.045979703345944 rpy=1.5707963267949 -1.5707963267949 0 -> xyz=0.0700000000000002 0 0.045979703345944 rpy=0 0 0
- joint FL_J3: axis 0 0 1 -> 1 0 0; origin xyz=0.318 0 0 rpy=0 0 0 -> xyz=0 0 0.318 rpy=0 0 0
- joint FR_J1: origin xyz=-0.1 0.05 0.20557 rpy=0 0 1.5708 -> xyz=-0.1 0.05 0.205567 rpy=0 0 0
- joint FR_J2: axis 0 0 -1 -> 1 0 0; origin xyz=0 0.07 0.04598 rpy=1.5708 -1.5708 0 -> xyz=-0.0700000000000002 0 0.045979703345944 rpy=0 0 0
- joint FR_J3: axis 0 0 1 -> -1 0 0; origin xyz=0.318 0 0 rpy=0 0 0 -> xyz=0 0 0.318 rpy=0 0 0

Commit message: urdf should be good this time... so close

File: urdf/Quad/urdf/Quad.urdf (robot description, URDF)
Before this commit: robot Quad, 13 links, 12 joints
Joints:
- joint BL_J1: origin xyz=0.1 0.05 -0.205567 rpy=0 0 0 -> xyz=0.1 0.05 -0.20557 rpy=0 0 0
- joint BR_J1: origin xyz=-0.1 0.0500000000000001 -0.205567 rpy=0 0 0 -> xyz=-0.1 0.05 -0.20557 rpy=0 0 0
- joint FL_J1: axis 0 0 0 -> 0 0 -1; origin xyz=0.1 0.05 0.205567 rpy=0 0 0 -> xyz=0.1 0.05 0.20557 rpy=0 0 0; type fixed -> continuous
- joint FR_J1: origin xyz=-0.1 0.05 0.205567 rpy=0 0 0 -> xyz=-0.1 0.05 0.20557 rpy=0 0 0

Commit message: this time for sure!

File: urdf/Quad/urdf/Quad.urdf (robot description, URDF)
Before this commit: robot Quad, 13 links, 12 joints
Links:
- link BR_Thigh: mass 0.179307876346527 -> 0.232342826148228
- link Body: mass 7.93838617368297 -> 7.96562277913682
- link FL_Thigh: mass 0.179307876346527 -> 0.232342826148228
Joints:
- joint BL_J1: origin xyz=0.1 0.05 -0.20557 rpy=0 0 0 -> xyz=0.1 0.05 -0.205567 rpy=0 0 0
- joint BR_J1: origin xyz=-0.1 0.05 -0.20557 rpy=0 0 0 -> xyz=-0.1 0.0500000000000001 -0.205567 rpy=0 0 0
- joint FL_J1: origin xyz=0.1 0.05 0.20557 rpy=0 0 0 -> xyz=0.1 0.05 0.205567 rpy=0 0 0
- joint FR_J1: origin xyz=-0.1 0.05 0.20557 rpy=0 0 0 -> xyz=-0.1 0.05 0.205567 rpy=0 0 0
