Commit message: There is some reset bug in quad jumpy still

File: isaac/IsaacGymEnvs/assets/urdf/Quad_Foot/urdf/Quad_Foot.urdf (robot description, URDF)
Before this commit: robot Quad_Foot, 17 links, 16 joints
Links:
- link Body: mass 7.8723215089476 -> 1.0

Commit message: Fixed the env reset bug. It learns better but i think the reward or observation need to be improved still.

File: isaac/IsaacGymEnvs/assets/urdf/Quad_Foot/urdf/Quad_Foot.urdf (robot description, URDF)
Before this commit: robot Quad_Foot, 17 links, 16 joints
Links:
- link BL_Hip: geometry visual mesh filename=../meshes/BL_Hip.STL
- link BR_Hip: geometry visual mesh filename=../meshes/BR_Hip.STL
- link FL_Hip: geometry visual mesh filename=../meshes/FL_Hip.STL
- link FR_Hip: geometry visual mesh filename=../meshes/FR_Hip.STL
Joints:
- joint BL_J2: limit (none) -> lower=-2.5 upper=2.5; type continuous -> revolute
- joint BL_J3: limit (none) -> lower=-3 upper=3; type continuous -> revolute
- joint BR_J2: limit (none) -> lower=-2.5 upper=2.5; type continuous -> revolute
- joint BR_J3: limit (none) -> lower=-3 upper=3; type continuous -> revolute
- joint FL_J2: limit (none) -> lower=-2.5 upper=2.5; type continuous -> revolute
- joint FL_J3: limit (none) -> lower=-3 upper=3; type continuous -> revolute
- joint FR_J2: limit (none) -> lower=-2.5 upper=2.5; type continuous -> revolute
- joint FR_J3: limit (none) -> lower=-3 upper=3; type continuous -> revolute

Commit message: Quad Walk Policy is working ok. I think i get better finally policies with goal oriented training as oppose to input oriented training... back to waypoints!

File: isaac/IsaacGymEnvs/assets/urdf/Quad_Foot/urdf/Quad_Foot.urdf (robot description, URDF)
Before this commit: robot Quad_Foot, 17 links, 16 joints
Joints:
- joint BL_J1: limit lower=0 upper=0 effort=0 velocity=0 -> lower=-0.5 upper=0.5 effort=0 velocity=0
- joint BR_J1: limit lower=0 upper=0 effort=0 velocity=0 -> lower=-0.5 upper=0.5 effort=0 velocity=0
- joint FL_J1: limit lower=0 upper=0 effort=0 velocity=0 -> lower=-0.5 upper=0.5 effort=0 velocity=0
- joint FR_J1: limit lower=0 upper=0 effort=0 velocity=0 -> lower=-0.5 upper=0.5 effort=0 velocity=0
