Commit message: Fixed the biped URDF after checking with isaac sim

File: urdf/Biped/urdf/Biped.urdf (robot description, URDF)
Before this commit: robot Biped, 9 links, 8 joints
Links:
- removed link FL_Hip
- removed link FL_Shin
- removed link FL_Thigh
- removed link FR_Hip
- removed link FR_Shin
- removed link FR_Thigh
- added link L_Hip, mass 0.244991798913576; collision mesh filename=package://Biped/meshes/L_Hip.STL; visual mesh filename=package://Biped/meshes/L_Hip.STL
- added link L_Shin, mass 0.0663666464185944; collision mesh filename=package://Biped/meshes/L_Shin.STL; visual mesh filename=package://Biped/meshes/L_Shin.STL
- added link L_Thigh, mass 0.246616840112844; collision mesh filename=package://Biped/meshes/L_Thigh.STL; visual mesh filename=package://Biped/meshes/L_Thigh.STL
- added link R_Hip, mass 0.244991783639153; collision mesh filename=package://Biped/meshes/R_Hip.STL; visual mesh filename=package://Biped/meshes/R_Hip.STL
- added link R_Shin, mass 0.0663666464185944; collision mesh filename=package://Biped/meshes/R_Shin.STL; visual mesh filename=package://Biped/meshes/R_Shin.STL
- added link R_Thigh, mass 0.229986631658005; collision mesh filename=package://Biped/meshes/R_Thigh.STL; visual mesh filename=package://Biped/meshes/R_Thigh.STL
- link Body: mass 3.8947264825535 -> 3.9263676397096
Joints:
- removed joint FL_J1
- removed joint FL_J2
- removed joint FL_J3
- removed joint FR_J1
- removed joint FR_J2
- removed joint FR_J3
- added joint L_J1: type revolute, parent Body, child L_Hip, origin xyz=-0.00556699999999997 0.1 0.05 rpy=0 0 0, axis 1 0 0, limit lower=-0.35 upper=0.35 effort=2 velocity=0
- added joint L_J2: type revolute, parent L_Hip, child L_Thigh, origin xyz=-0.045979703345944 0.07 0 rpy=0 0 0, axis 0 -1 0, limit lower=-2.8 upper=2.8 effort=2 velocity=0
- added joint L_J3: type revolute, parent L_Thigh, child L_Shin, origin xyz=-0.218 0 0 rpy=0 0 0, axis 0 1 0, limit lower=-2.8 upper=2.8 effort=2 velocity=0
- added joint R_J1: type revolute, parent Body, child R_Hip, origin xyz=-0.00556700000000009 -0.1 0.05 rpy=0 0 0, axis 1 0 0, limit lower=-0.35 upper=0.35 effort=2 velocity=0
- added joint R_J2: type revolute, parent R_Hip, child R_Thigh, origin xyz=-0.045979703345944 -0.07 0 rpy=0 0 0, axis 0 1 0, limit lower=-2.8 upper=2.8 effort=2 velocity=0
- added joint R_J3: type revolute, parent R_Thigh, child R_Shin, origin xyz=-0.218 0 0 rpy=0 0 0, axis 0 -1 0, limit lower=-2.8 upper=2.8 effort=2 velocity=0
- joint WheelX: origin xyz=-0.07 0 0.05 rpy=0 0 0 -> xyz=-0.0699999999999999 0 0.05 rpy=0 0 0
- joint WheelY: origin xyz=0.020147 0 0.05 rpy=0 0 0 -> xyz=0.020147207668468 0 0.05 rpy=0 0 0
