File: kicad/MotorDriver/DRV8323RS.kicad_sch (KiCad schematic)
At the start: 72 parts, among them J1 Conn_01x02_Socket, J2 Conn_01x03_Socket, U1 DRV8323RSRGZR, U2 CSD88599Q5DC, U3 CSD88599Q5DC, U5 CSD88599Q5DC

Commit message: Updated the planetary gearbox design. It is much better with retaining rings and bearing support. 95% done with the PCB routing. Need to just do a final routing check and i think I can put the order in
Parts:
- removed C3, C4: 330uF, Capacitor_SMD:C_0603_1608Metric, symbol Device:C
- removed TP1, TP4, TP7: TestPoint, TestPoint:TestPoint_Pad_D2.5mm, symbol Connector:TestPoint
- added C26, C27: 220uF, TylerLib:CHEMI-HA0, symbol TylerLib:EMVY350ADA221MHA0G
- added R5: 330, Resistor_SMD:R_0603_1608Metric, symbol Device:R
- C10, C12, C2, R1, R10, R12, R13, R2, R9: now not fitted
- C13, C19: footprint Capacitor_SMD:C_0603_1608Metric -> Capacitor_SMD:C_1210_3225Metric
- C24: footprint Capacitor_SMD:C_0603_1608Metric -> Capacitor_SMD:C_0805_2012Metric
- D4: value MBR1H100SFT3G -> NRVB1H100SFT3G; footprint Diode_SMD:D_MELF -> TylerLib:DIODE_SOD123LF_2P9X1P8_ONS
- L1: footprint Inductor_SMD:L_0603_1608Metric -> TylerLib:IND_VLS3015CX-150M-1
- R11, R14, R3: footprint Resistor_SMD:R_0603_1608Metric -> Resistor_SMD:R_2512_6332Metric
Connections:
- net SEN.SOA is gone; now on net SOA: U1.25 (SOA)
- net SEN.SOB is gone; now on net SOB: U1.24 (SOB)
- net SEN.SOC is gone; now on net SOC: U1.23 (SOC)
- net VSENVM is gone; now on net SEN.VSENVM: U4.6 (D1-)
- net GND: now also C26.2, C27.2, R5.2; no longer D1.1 (K)
- net Vdrive: now also J1.1 (Pin_1), R4.1, C26.1, C27.1
- net ISENA renamed SEN.ISENA
- net ISENB renamed SEN.ISENB
- net ISENC renamed SEN.ISENC
- net VSENA: no longer names the net of U4.1 (D1+)
- net VSENB: no longer names the net of U4.3 (D2+)
- net VSENC: no longer names the net of U4.4 (D2-)
- new net: D1.1 (K), R5.1
Other:
- note added: "SEN.VSENA"
- note added: "SEN.VSENB"
- note added: "SEN.VSENC"
- moved on the sheet: D1

Commit message: PCB ordered
Parts:
- removed C14, C18, C23: 0.1uF, Capacitor_SMD:C_0603_1608Metric, symbol Device:C
- added C4 (x3): 0.1uF, Capacitor_SMD:C_0603_1608Metric, symbol Device:C
- C1, C11: value 0.01 uF -> 10000pF
- C9: value 0.01 uF -> 10000 pF
- D1: value LED -> BlueLED
- D3: value LED -> RedLED
- U4: value ~ -> TPD4S009DCKR
Connections:
- net +3.3V: now also C4.1
- net GND: now also C4.2, C4.2
- net Vdrive: now also C4.1
- net at D4.1 (K), L1.1, U1.45 (SW): now also C4.2
- net at U1.44 (CB): now also C4.1

Commit message: Working on some of the solidworks model, new urdf, working on the motor drive board a little
Parts:
- added TP2 (x6): TestPoint, TestPoint:TestPoint_Pad_D1.0mm, symbol Connector:TestPoint
- TP2, TP3, TP5, TP6, TP8, TP9: footprint TestPoint:TestPoint_Pad_D2.5mm -> TestPoint:TestPoint_Pad_D1.0mm
Connections:
- net DRV.INHA: now also TP2.1
- net DRV.INHB: now also TP2.1
- net DRV.INHC: now also TP2.1
- net DRV.INLA: now also TP2.1
- net DRV.INLB: now also TP2.1
- net DRV.INLC: now also TP2.1
Changed lines of the file:
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@@
     (stroke (width 0) (type default))
   )
-  (wire (pts (xy 76.2 97.79) (xy 86.995 97.79))
+  (wire (pts (xy 74.295 97.79) (xy 86.995 97.79))
     (stroke (width 0) (type default))
   )
@@
     (stroke (width 0) (type default))
   )
-  (wire (pts (xy 76.2 87.63) (xy 86.995 87.63))
+  (wire (pts (xy 78.105 87.63) (xy 86.995 87.63))
     (stroke (width 0) (type default))
   )
@@
     (stroke (width 0) (type default))
   )
-  (wire (pts (xy 76.2 105.41) (xy 86.995 105.41))
+  (wire (pts (xy 74.295 105.41) (xy 86.995 105.41))
     (stroke (width 0) (type default))
   )
@@
     (effects (font (size 1.27 1.27)) (justify left bottom))
   )
-  (label "DRV.INHA" (at 76.2 87.63 0) (fields_autoplaced)
+  (label "DRV.INHA" (at 78.105 87.63 0) (fields_autoplaced)
     (effects (font (size 1.27 1.27)) (justify left bottom))
   )
@@
       (effects (font (size 1.27 1.27)) (justify left) hide)
     )
-    (property "Footprint" "TestPoint:TestPoint_Pad_D2.5mm" (at 284.48 69.85 0)
+    (property "Footprint" "TestPoint:TestPoint_Pad_D1.0mm" (at 284.48 69.85 0)
       (effects (font (size 1.27 1.27)) hide)
     )
@@
     )
   )
+  (symbol (lib_id "Connector:TestPoint") (at 76.2 102.87 90) (unit 1)
+    (in_bom yes) (on_board yes) (dnp no)
+    (property "Reference" "TP2" (at 71.12 104.14 0)
+      (effects (font (size 1.27 1.27)) (justify left))
+    )
+    (property "Value" "TestPoint" (at 74.168 100.33 0)
+      (effects (font (size 1.27 1.27)) (justify left) hide)
+    )
+    (property "Footprint" "TestPoint:TestPoint_Pad_D1.0mm" (at 76.2 97.79 0)
+      (effects (font (size 1.27 1.27)) hide)
+    )
+    (property "Datasheet" "~" (at 76.2 97.79 0)
+      (effects (font (size 1.27 1.27)) hide)
+    )
+    (pin "1")
+    (instances
+      (project "MotorDriver"
+        (path "/1fa4c72f-b85f-4d78-9713-26aa572ca2e5"
+          (reference "TP2") (unit 1)
+        )
+        (path "/1fa4c72f-b85f-4d78-9713-26aa572ca2e5/c363089b-1b0b-4509-af19-a6f84e71682e"
+          (reference "TP15") (unit 1)
+        )
+      )
+    )
+  )
   (symbol (lib_id "Connector:TestPoint") (at 347.98 63.5 0) (unit 1)
     (in_bom yes) (on_board yes) (dnp no)
@@
       (effects (font (size 1.27 1.27)) (justify left) hide)
     )
-    (property "Footprint" "TestPoint:TestPoint_Pad_D2.5mm" (at 353.06 63.5 0)
+    (property "Footprint" "TestPoint:TestPoint_Pad_D1.0mm" (at 353.06 63.5 0)
       (effects (font (size 1.27 1.27)) hide)
     )
@@
     )
   )
+  (symbol (lib_id "Connector:TestPoint") (at 78.105 87.63 90) (unit 1)
+    (in_bom yes) (on_board yes) (dnp no)
+    (property "Reference" "TP2" (at 73.025 88.9 0)
+      (effects (font (size 1.27 1.27)) (justify left))
+    )
+    (property "Value" "TestPoint" (at 76.073 85.09 0)
+      (effects (font (size 1.27 1.27)) (justify left) hide)
+    )
+    (property "Footprint" "TestPoint:TestPoint_Pad_D1.0mm" (at 78.105 82.55 0)
+      (effects (font (size 1.27 1.27)) hide)
+    )
+    (property "Datasheet" "~" (at 78.105 82.55 0)
+      (effects (font (size 1.27 1.27)) hide)
+    )
+    (pin "1")
+    (instances
+      (project "MotorDriver"
+        (path "/1fa4c72f-b85f-4d78-9713-26aa572ca2e5"
+          (reference "TP2") (unit 1)
+        )
+        (path "/1fa4c72f-b85f-4d78-9713-26aa572ca2e5/c363089b-1b0b-4509-af19-a6f84e71682e"
+          (reference "TP19") (unit 1)
+        )
+      )
+    )
+  )
   (symbol (lib_id "Device:R") (at 190.5 133.985 0) (mirror y) (unit 1)
     (in_bom yes) (on_board yes) (dnp no)
@@
       (effects (font (size 1.27 1.27)) (justify left) hide)
     )
-    (property "Footprint" "TestPoint:TestPoint_Pad_D2.5mm" (at 284.48 62.23 0)
+    (property "Footprint" "TestPoint:TestPoint_Pad_D1.0mm" (at 284.48 62.23 0)
       (effects (font (size 1.27 1.27)) hide)
     )
@@
     )
   )
+  (symbol (lib_id "Connector:TestPoint") (at 76.2 90.17 90) (unit 1)
+    (in_bom yes) (on_board yes) (dnp no)
+    (property "Reference" "TP2" (at 71.12 91.44 0)
+      (effects (font (size 1.27 1.27)) (justify left))
+    )
+    (property "Value" "TestPoint" (at 74.168 87.63 0)
+      (effects (font (size 1.27 1.27)) (justify left) hide)
+    )
+    (property "Footprint" "TestPoint:TestPoint_Pad_D1.0mm" (at 76.2 85.09 0)
+      (effects (font (size 1.27 1.27)) hide)
+    )
+    (property "Datasheet" "~" (at 76.2 85.09 0)
+      (effects (font (size 1.27 1.27)) hide)
+    )
+    (pin "1")
+    (instances
+      (project "MotorDriver"
+        (path "/1fa4c72f-b85f-4d78-9713-26aa572ca2e5"
+          (reference "TP2") (unit 1)
+        )
+        (path "/1fa4c72f-b85f-4d78-9713-26aa572ca2e5/c363089b-1b0b-4509-af19-a6f84e71682e"
+          (reference "TP18") (unit 1)
+        )
+      )
+    )
+  )
   (symbol (lib_id "Device:NetTie_2") (at 420.37 67.31 0) (unit 1)
     (in_bom no) (on_board yes) (dnp no) (fields_autoplaced)
@@
     )
   )
+  (symbol (lib_id "Connector:TestPoint") (at 74.295 105.41 90) (unit 1)
+    (in_bom yes) (on_board yes) (dnp no)
+    (property "Reference" "TP2" (at 69.215 106.68 0)
+      (effects (font (size 1.27 1.27)) (justify left))
+    )
+    (property "Value" "TestPoint" (at 72.263 102.87 0)
+      (effects (font (size 1.27 1.27)) (justify left) hide)
+    )
+    (property "Footprint" "TestPoint:TestPoint_Pad_D1.0mm" (at 74.295 100.33 0)
+      (effects (font (size 1.27 1.27)) hide)
+    )
+    (property "Datasheet" "~" (at 74.295 100.33 0)
+      (effects (font (size 1.27 1.27)) hide)
+    )
+    (pin "1")
+    (instances
+      (project "MotorDriver"
+        (path "/1fa4c72f-b85f-4d78-9713-26aa572ca2e5"
+          (reference "TP2") (unit 1)
+        )
+        (path "/1fa4c72f-b85f-4d78-9713-26aa572ca2e5/c363089b-1b0b-4509-af19-a6f84e71682e"
+          (reference "TP14") (unit 1)
+        )
+      )
+    )
+  )
   (symbol (lib_id "power:GND") (at 345.44 125.73 0) (unit 1)
     (in_bom yes) (on_board yes) (dnp no) (fields_autoplaced)
@@
     )
   )
+  (symbol (lib_id "Connector:TestPoint") (at 74.295 97.79 90) (unit 1)
+    (in_bom yes) (on_board yes) (dnp no)
+    (property "Reference" "TP2" (at 69.215 99.06 0)
+      (effects (font (size 1.27 1.27)) (justify left))
+    )
+    (property "Value" "TestPoint" (at 72.263 95.25 0)
+      (effects (font (size 1.27 1.27)) (justify left) hide)
+    )
+    (property "Footprint" "TestPoint:TestPoint_Pad_D1.0mm" (at 74.295 92.71 0)
+      (effects (font (size 1.27 1.27)) hide)
+    )
+    (property "Datasheet" "~" (at 74.295 92.71 0)
+      (effects (font (size 1.27 1.27)) hide)
+    )
+    (pin "1")
+    (instances
+      (project "MotorDriver"
+        (path "/1fa4c72f-b85f-4d78-9713-26aa572ca2e5"
+          (reference "TP2") (unit 1)
+        )
+        (path "/1fa4c72f-b85f-4d78-9713-26aa572ca2e5/c363089b-1b0b-4509-af19-a6f84e71682e"
+          (reference "TP16") (unit 1)
+        )
+      )
+    )
+  )
   (symbol (lib_id "power:Vdrive") (at 53.34 53.34 0) (unit 1)
     (in_bom yes) (on_board yes) (dnp no) (fields_autoplaced)
@@
       (effects (font (size 1.27 1.27)) (justify left) hide)
     )
-    (property "Footprint" "TestPoint:TestPoint_Pad_D2.5mm" (at 422.91 63.5 0)
+    (property "Footprint" "TestPoint:TestPoint_Pad_D1.0mm" (at 422.91 63.5 0)
       (effects (font (size 1.27 1.27)) hide)
     )
@@
       (effects (font (size 1.27 1.27)) (justify left) hide)
     )
-    (property "Footprint" "TestPoint:TestPoint_Pad_D2.5mm" (at 422.91 71.12 0)
+    (property "Footprint" "TestPoint:TestPoint_Pad_D1.0mm" (at 422.91 71.12 0)
       (effects (font (size 1.27 1.27)) hide)
     )
@@
       (effects (font (size 1.27 1.27)) (justify left) hide)
     )
-    (property "Footprint" "TestPoint:TestPoint_Pad_D2.5mm" (at 353.06 71.12 0)
+    (property "Footprint" "TestPoint:TestPoint_Pad_D1.0mm" (at 353.06 71.12 0)
       (effects (font (size 1.27 1.27)) hide)
     )
@@
         )
       )
+    )
+  )
+  (symbol (lib_id "Connector:TestPoint") (at 76.2 95.25 90) (unit 1)
+    (in_bom yes) (on_board yes) (dnp no)
+    (property "Reference" "TP2" (at 71.12 96.52 0)
+      (effects (font (size 1.27 1.27)) (justify left))
+    )
+    (property "Value" "TestPoint" (at 74.168 92.71 0)
+      (effects (font (size 1.27 1.27)) (justify left) hide)
+    )
+    (property "Footprint" "TestPoint:TestPoint_Pad_D1.0mm" (at 76.2 90.17 0)
+      (effects (font (size 1.27 1.27)) hide)
+    )
+    (property "Datasheet" "~" (at 76.2 90.17 0)
+      (effects (font (size 1.27 1.27)) hide)
+    )
+    (pin "1")
+    (instances
+      (project "MotorDriver"
+        (path "/1fa4c72f-b85f-4d78-9713-26aa572ca2e5"
+          (reference "TP2") (unit 1)
+        )
+        (path "/1fa4c72f-b85f-4d78-9713-26aa572ca2e5/c363089b-1b0b-4509-af19-a6f84e71682e"
+          (reference "TP17") (unit 1)
+        )
+      )
