File: kicad/MotorDriver/stm32f446.kicad_sch (KiCad schematic)
At the start: 34 parts, among them J1 Conn_01x03_Pin, J2 Conn_01x06_Pin, J3 Conn_01x02_Pin, U2 ATA6560-GAQW, U8 STM32F446RETx, Y1 8.000MHZ

Commit message: Pushing before the drive to Boston...
Parts:
- removed Y1: 8.000MHZ, TylerLib:XTAL_ABLS2-8.000MHZ-B1U-T, symbol TylerLib:ABLS2-8.000MHZ-B1U-T
- added Y2: ABL-8.000MHZ-B1U-T, TylerLib:XTAL_ABL-8.000MHZ-B1U-T, symbol TylerLib:ABL-8.000MHZ-B1U-T
Connections:
- net +3.3V: no longer C4.2
- net at C4.2, R19.2: now also Y2.1
- net at C4.2, R19.2: now also Y2.2
- net VDDA: now reaches L1.1, U8.13 (VDDA)
- net VDDA: now also C4.2
Other:
- moved on the sheet: L1

Commit message: Updated the planetary gearbox design. It is much better with retaining rings and bearing support. 95% done with the PCB routing. Need to just do a final routing check and i think I can put the order in
Parts:
- removed C4: 4.7uF, Capacitor_SMD:C_0603_1608Metric, symbol Device:C
- removed C4 (x2): 100nF, Capacitor_SMD:C_0603_1608Metric, symbol Device:C
- removed R22: 100, Resistor_SMD:R_0603_1608Metric, symbol Device:R
- removed R22: 4.7k, Resistor_SMD:R_0603_1608Metric, symbol Device:R
- removed S1, S2: TS04-66-75-BK-160-SMT, TylerLib:SW_TS04-66-75-BK-160-SMT, symbol TylerLib:TS04-66-75-BK-160-SMT
- removed TP1 (x3): TestPoint, TestPoint:TestPoint_Pad_D2.5mm, symbol Connector:TestPoint
- added C19: 4.7uF, Capacitor_SMD:C_1210_3225Metric, symbol Device:C
- J2: footprint Connector_PinHeader_2.54mm:PinHeader_2x03_P2.54mm_Vertical -> Connector_PinHeader_2.54mm:PinHeader_1x06_P2.54mm_Vertical
Connections:
- net DRV.INHA: no longer U8.34 (PB13)
- net DRV.INHB: no longer U8.35 (PB14)
- net DRV.INHC: no longer U8.36 (PB15)
- net DRV.INLA: now also U8.34 (PB13)
- net DRV.INLB: now also U8.35 (PB14)
- net DRV.INLC: now also U8.36 (PB15)
- net GND: now also C19.1
- net at U8.30 (VCAP_1): now also C19.2
- net CLK_P: now reaches R19.1, U8.5 (PH0)
- net CLK_N: now reaches R19.1, U8.6 (PH1)
- net SEN.SOA renamed SEN.ISENA
- net SEN.SOB renamed SEN.ISENB
- net SEN.SOC renamed SEN.ISENC

Commit message: PCB ordered
Parts:
- removed C4 (x5): 100nF, Capacitor_SMD:C_0603_1608Metric, symbol Device:C
- removed D5, D6, D7: LED, LED_SMD:LED_0603_1608Metric, symbol Device:LED
- removed R19 (x2): 80, Resistor_SMD:R_0603_1608Metric, symbol Device:R
- added C4 (x5): 0.1uF, Capacitor_SMD:C_0603_1608Metric, symbol Device:C
- added U9: 150066M153000, TylerLib:CHIP_M153000_WRE, symbol TylerLib:150066M153000
- C4: value 100nF -> 0.1uF
- R20: value 1k -> 330
Connections:
- net +3.3V: now also C4.2, C4.2, C4.2, C4.2, U9.4
- net CLK_N: now also C4.2, Y2.1
- net CLK_P: now also C4.2, Y2.2
- net GND: now also C4.1, C4.1, C4.1, C4.1, C4.1; no longer R20.2, R22.2, R23.2
- net VDDA: now also C4.2
- net at R23.1: now also U8.39 (PC8)
- net at R22.1: now also U8.38 (PC7)
- net at R20.1: now also U8.37 (PC6)
- new net: R22.2, U9.2
- new net: R23.2, U9.1
- new net: R20.2, U9.3
Other:
- moved on the sheet: R20, R22, R23

Commit message: Working on some of the solidworks model, new urdf, working on the motor drive board a little
Parts:
- removed Y2: ABL-8.000MHZ-B1U-T, TylerLib:XTAL_ABL-8.000MHZ-B1U-T, symbol TylerLib:ABL-8.000MHZ-B1U-T
- added Y1: 406I35D08M00000, TylerLib:XTAL_406I35D08M00000, symbol TylerLib:406I35D08M00000
Connections:
- net CLK_N: now also Y1.3
- net CLK_P: now also Y1.1
- net GND: now also Y1.2 (GND), Y1.4 (GND__1)
Other:
- moved on the sheet: C4
