File: kicad/MotorDriver/MotorDriver.kicad_pcb (KiCad board)
At the start: 4 copper layers, 59 x 55.3 mm, 97 parts, among them J1 Conn_01x03_Pin, J2 Conn_01x06_Pin, J3 Conn_01x02_Pin, J4 Conn_01x02_Socket, J5 Conn_01x03_Socket, U1 STM32F446RETx, U2 ATA6560-GAQW, U3 AS5147U, U4 DRV8323RSRGZR, U5 CSD88599Q5DC, U6 CSD88599Q5DC, U7 TPD4S009DCKR, U8 CSD88599Q5DC, U9 150066M153000, Y1 406I35D08M00000

Commit message: Adding STM32 Motor Drive Stuff for testing
Parts:
- added ?: LOGO, LOGO, F.Cu at (83.8, 134.6)
- moved C6 1.47 mm to (81.5, 136.2), turned to 90 degrees
- moved C10 0.73 mm to (78.2, 135.8), turned to 0 degrees
- moved C5 0.20 mm to (77.7, 149.5)
- turned U7 to 0 degrees
Routing:
- net +3.3V: track 56.0 -> 53.8 mm
- net /Microcontroller/SEN.VSENVM: track 29.5 -> 27.5 mm
- net /Microcontroller/UART_TX: track 27.9 -> 28.5 mm
- net /Microcontroller/UART_RX: track 28.4 -> 28.9 mm
