Commit message: Set the JumpRig training environment up... time to learn

File: isaac/IsaacGymEnvs/assets/urdf/Biped/urdf/Biped.urdf (robot description, URDF)
Before this commit: robot Biped, 9 links, 8 joints
Joints:
- removed joint WheelX
- removed joint WheelY
- added joint Wheel_X: type continuous, parent Body, child ReactionWheelX, origin xyz=-0.0699999999999999 0 0.05 rpy=0 0 0, axis 1 0 0
- added joint Wheel_Y: type continuous, parent Body, child ReactionWheelY, origin xyz=0.020147207668468 0 0.05 rpy=0 0 0, axis 0 1 0
