Commit message: Working on some wonky collision physics. I think i need to make the foot a fixed joint so it can have its own collision mesh...

File: isaac/IsaacGymEnvs/assets/urdf/JumpRig2/urdf/JumpRig2.urdf (robot description, URDF)
Before this commit: robot JumpRig2, 4 links, 3 joints
Links:
- link Base: geometry visual mesh filename=../meshes/Base.STL
- link Carriage: geometry visual mesh filename=../meshes/Carriage.STL
- link Hip: geometry visual mesh filename=../meshes/Hip.STL
Joints:
- joint Prismatic1: limit lower=0.0 upper=0.6 effort=0 velocity=0 -> lower=-0.3 upper=0.6 effort=0 velocity=0
