Commit message: Updated the jump rig 2 urdf to have a seperate collision mesh for the foot element

File: urdf/JumpRig2/urdf/JumpRig2.urdf (robot description, URDF)
Before this commit: robot JumpRig2, 4 links, 3 joints
Links:
- added link Foot, mass 0.0290279405926851; collision mesh filename=package://JumpRig2/meshes/Foot.STL; visual mesh filename=package://JumpRig2/meshes/Foot.STL
- link Base: mass 1.1645 -> 1.16451700934069
- link Carriage: mass 0.43811 -> 0.438107006723366
- link Hip: mass 0.10809 -> 0.108085294122534
- link Knee: mass 0.29663 -> 0.267605307693932
Joints:
- added joint Fixed1: type fixed, parent Knee, child Foot, origin xyz=0.061 -0.0123 -0.3 rpy=0 0 0, axis 0 0 0
- joint Prismatic1: axis 0 0 1 -> 0 0 -1
- joint Revolute1: axis 0 1 0 -> 0 -1 0
- joint Revolute2: axis 0 1 0 -> 0 -1 0

Commit message: Added another collision mesh for the shin... still working out the wonky physics... it seems to be related to an self interaction of collision mesh potentially

File: urdf/JumpRig2/urdf/JumpRig2.urdf (robot description, URDF)
Before this commit: robot JumpRig2, 5 links, 4 joints
Links:
- added link Shin, mass 0.102797649052896; collision mesh filename=package://JumpRig2/meshes/Shin.STL; visual mesh filename=package://JumpRig2/meshes/Shin.STL
- link Knee: mass 0.267605307693932 -> 0.164807658641037
Joints:
- added joint Fixed2: type fixed, parent Shin, child Foot, origin xyz=0 0 -0.300000000000001 rpy=0 0 0, axis 0 0 0
- joint Fixed1: child Foot -> Shin; origin xyz=0.061 -0.0123 -0.3 rpy=0 0 0 -> xyz=0.061 -0.0123 0 rpy=0 0 0
- joint Prismatic1: axis 0 0 -1 -> 0 0 1; limit lower=0 upper=10 effort=0 velocity=0 -> lower=-0.15 upper=0.6 effort=0 velocity=0
- joint Revolute1: axis 0 -1 0 -> 0 1 0
- joint Revolute2: axis 0 -1 0 -> 0 1 0
